File: pcb/Fuente_para_protoboard.kicad_pcb (KiCad board)
At the start: 2 copper layers, 56 x 39 mm, 21 parts, among them J1 Conn_01x04, J2 Conn_01x02, J3 Conn_01x02, J4 Conn_01x02, J5 USB_A, J6 Conn_01x04, J7 Conn_01x02, J8 Conn_01x02, J9 Conn_02x04_Odd_Even, SW1 GPBS-850N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

Commit message: Correcciones realizadas
Other:
- board text added: "Réplica"
