File: pcb/Fuente_para_protoboard.sch (KiCad schematic (older format))
At the start: 21 parts, among them J1 Conn_01x04, J2 Conn_01x02, J3 Conn_01x02, J4 Conn_01x02, J5 USB_A, J6 Conn_01x04, J7 Conn_01x02, J8 Conn_01x02, J9 Conn_02x04_Odd_Even, SW1 GPBS-850N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

Commit message: Huellas, posicionamiento, modelos 3D y ruteo
Parts:
- C1: footprint (none) -> Capacitor_THT:CP_Radial_D6.3mm_P2.50mm
- C2, C3, C4: footprint (none) -> Capacitor_SMD:C_0805_2012Metric
- D1: footprint (none) -> Diode_SMD:D_SMA
- D2: footprint (none) -> LED_THT:LED_D3.0mm
- H1, H2: footprint (none) -> MountingHole:MountingHole_2.7mm
- J1, J6: footprint (none) -> Connector_PinHeader_2.54mm:PinHeader_1x04_P2.54mm_Vertical
- J2, J3, J7, J8: footprint (none) -> Connector_PinHeader_2.54mm:PinHeader_1x02_P2.54mm_Vertical
- J4: footprint (none) -> Connector_BarrelJack:BarrelJack_CUI_PJ-063AH_Horizontal
- J5: footprint (none) -> Connector_USB:USB_A_Molex_67643_Horizontal; symbol Connector:USB_A -> Fuente_para_protoboard-rescue:USB_A-Connector
- J9: footprint (none) -> Connector_PinHeader_2.54mm:PinHeader_2x04_P2.54mm_Vertical
- R1: footprint (none) -> Resistor_SMD:R_0805_2012Metric
- SW1: footprint (none) -> pcb:GPBS850NR1
- U1, U2: footprint Package_TO_SOT_SMD:SOT-223-3_TabPin2 -> digikey-footprints:SOT-223
Connections:
- net +3V3: now also J9.2 (Pin_2), J9.4 (Pin_4); no longer J9.6 (Pin_6), J9.8 (Pin_8)
- net +5V: now also J9.6 (Pin_6), J9.8 (Pin_8); no longer J9.2 (Pin_2), J9.4 (Pin_4)
- net Earth: now also J5.5 (Shield)
- no-connect marks 5 -> 4

Commit message: Correcciones realizadas
Parts:
- D1: Catalog (none) -> https://www.digikey.com/en/products/detail/diotec-semicondu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
- J5: Catalog (none) -> https://www.digikey.com/en/products/detail/gct/USB1135-15-9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
- U1: Catalog (none) -> https://www.digikey.com/en/products/detail/texas-instrument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
Changed lines of the file:
@@
 F 1 "USB_A" H 3300 2750 50  0000 C CNN
 F 2 "Connector_USB:USB_A_Molex_67643_Horizontal" H 3800 2850 50  0001 C CNN
-F 3 " ~" H 3800 2850 50  0001 C CNN
+F 3 "https://media.digikey.com/pdf/Data%20Sheets/GCT%20PDFs/USB1130-USB1135.pdf" H 3800 2850 50  0001 C CNN
+F 4 "https://www.digikey.com/en/products/detail/gct/USB1135-15-9-L-B/13545895" H 3650 2900 50  0001 C CNN "Catalog"
 	1    3650 2900
 	1    0    0    -1
@@
 F 1 "M7" H 5500 1900 50  0000 C CNN
 F 2 "Diode_SMD:D_SMA" H 5500 1800 50  0001 C CNN
-F 3 "~" H 5500 1800 50  0001 C CNN
+F 3 "https://diotec.com/tl_files/diotec/files/pdf/datasheets/m1.pdf" H 5500 1800 50  0001 C CNN
+F 4 "https://www.digikey.com/en/products/detail/diotec-semiconductor/M7/13155808" H 5500 1800 50  0001 C CNN "Catalog"
 	1    5500 1800
 	-1   0    0    1
@@
 F 2 "digikey-footprints:SOT-223" H 6400 2000 50  0001 C CNN
 F 3 "http://www.advanced-monolithic.com/pdf/ds1117.pdf" H 6500 1550 50  0001 C CNN
+F 4 "https://www.digikey.com/en/products/detail/texas-instruments/LM1117MPX-5-0-NOPB/366734" H 6400 1800 50  0001 C CNN "Catalog"
 	1    6400 1800
 	1    0    0    -1
@@
 F 1 "AMS1117-3.3" H 7650 1951 50  0000 C CNN
 F 2 "digikey-footprints:SOT-223" H 7650 2000 50  0001 C CNN
-F 3 "http://www.advanced-monolithic.com/pdf/ds1117.pdf" H 7750 1550 50  0001 C CNN
+F 3 "https://www.digikey.com/en/products/detail/texas-instruments/LM1117MPX-3-3-NOPB/366733" H 7750 1550 50  0001 C CNN
 	1    7650 1800
 	1    0    0    -1
@@
 	7650 2100 7650 2450
 Wire Wire Line
-	5350 3400 5350 3600
+	5350 3400 5350 3550
 Wire Wire Line
 	6100 3550 6100 3600
@@
 	1    0    0    -1
 $EndComp
+$Comp
+L power:PWR_FLAG #FLG0104
+U 1 1 611AA4B9
+P 5400 3550
+F 0 "#FLG0104" H 5400 3625 50  0001 C CNN
+F 1 "PWR_FLAG" V 5400 3678 50  0000 L CNN
+F 2 "" H 5400 3550 50  0001 C CNN
+F 3 "~" H 5400 3550 50  0001 C CNN
+	1    5400 3550
+	0    1    1    0
+$EndComp
+Wire Wire Line
+	5400 3550 5350 3550
+Connection ~ 5350 3550
+Wire Wire Line
+	5350 3550 5350 3600
 $EndSCHEMATC
